File: controller/controller.brd (EAGLE design)
At the start: 101.6 x 53.3 mm, 22 parts

Commit message: test with timer
Connections:
- new net MA': PCB1.7
Changed lines of the file:
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@@
 <wire x1="32.385" y1="25.019" x2="32.639" y2="24.765" width="0.6096" layer="16"/>
+</signal>
+<signal name="MA'">
+<contactref element="PCB1" pad="7"/>
 </signal>
 </signals>
