File: driver/driver.sch (EAGLE design)
At the start: 38 parts, among them IC1 7805TV, IC2 7806T, Q1 IRF530, Q10 TIP31C, Q2 IRF9530, Q3 IRF530, Q4 IRF9530, Q5 IRF530, Q6 IRF9530, Q7 IRF530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

Commit message: test with timer
Changed lines of the file:
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@@
 <wire x1="66.04" y1="48.26" x2="66.04" y2="50.8" width="0.1524" layer="91"/>
 <label x="68.58" y="40.64" size="1.778" layer="95"/>
+<label x="63.5" y="45.72" size="1.778" layer="95"/>
 </segment>
 <segment>
